File: pcbs/programming_shield/shield/shield.sch (KiCad schematic (older format))
At the start: 8 parts, among them P1 Power, P2 Analog, P3 Digital, P4 Digital, P5 CONN_01X01, P6 CONN_01X01, P7 CONN_01X01, P8 CONN_01X01

Commit message: produced PCBs, dropped baudrate, removed on-board dynamic address selection - decoder must now be configured via programmer!
Parts:
- removed P5, P6, P7, P8: CONN_01X01, Socket_Arduino_Uno:Arduino_1pin, symbol Connector_Generic:Conn_01x01
- added D1: 1N4001, Diode_THT:D_DO-41_SOD81_P3.81mm_Vertical_KathodeUp, symbol Diode:1N4001
- added J1, J2: RJ45_LED, customs:RND_RJ45_LED, symbol Connector:RJ45_LED
- added J3: AVR-ISP-6, Connector_PinSocket_2.54mm:PinSocket_2x03_P2.54mm_Vertical, symbol Connector:AVR-ISP-6
- added OC1, OC2: CNY74-2H, Package_DIP:DIP-8_W7.62mm_LongPads, symbol custom:CNY74-2H
- added R1, R2, R3, R4, R5, R6, R7, R8, R9: R, Resistor_SMD:R_0603_1608Metric, symbol Device:R
- added U1: MAX489E, Package_SO:SOIC-14_3.9x8.7mm_P1.27mm, symbol Interface_UART:MAX489E
Connections:
- net labels added: 5V, sense+, sense+B, sense-, sense-B
- wire segments 38 -> 89
- no-connect marks 5 -> 1
