File: pcbs/programming_shield/shield/shield.kicad_pcb (KiCad board)
At the start: 2 copper layers, 52.7 x 53.3 mm, 20 parts, among them J1 RJ45_LED, J2 RJ45_LED, J3 AVR-ISP-6, P1 Power, P2 Analog, P3 Digital, P4 Digital, U1 MAX489E

Commit message: revision b of boards
Parts:
- removed the J2 at (165.0, 109.2)
- removed OC1, OC2: CNY74-2H, Package_DIP:DIP-8_W7.62mm_LongPads
- added C1: 10pF, Capacitor_SMD:C_0603_1608Metric, F.Cu at (146.7, 104.2)
- added C2: 10pF, Capacitor_SMD:C_0603_1608Metric, F.Cu at (142.8, 109.1)
- added C3: 100nF, Capacitor_THT:C_Disc_D3.0mm_W2.0mm_P2.50mm, F.Cu at (140.8, 95.9)
- added C4: 100nF, Capacitor_THT:C_Disc_D3.0mm_W2.0mm_P2.50mm, F.Cu at (140.8, 98.3)
- added D10: LED, LED_SMD:LED_0603_1608Metric, F.Cu at (172.0, 115.1)
- added D2: BAT54CW, Package_TO_SOT_SMD:SOT-23, F.Cu at (145.9, 99.5)
- added D3: LED, LED_SMD:LED_0603_1608Metric, F.Cu at (172.6, 84.5)
- added D4: LED, LED_SMD:LED_0603_1608Metric, F.Cu at (174.5, 84.5)
- added D5: LED, LED_SMD:LED_0603_1608Metric, F.Cu at (140.6, 84.2)
- added D6: LED, LED_SMD:LED_0603_1608Metric, F.Cu at (143.1, 84.2)
- added D7: LED, LED_SMD:LED_0603_1608Metric, F.Cu at (138.0, 84.2)
- added D8: LED, LED_SMD:LED_0603_1608Metric, F.Cu at (158.6, 114.4)
- added D9: LED, LED_SMD:LED_0603_1608Metric, F.Cu at (135.5, 84.2)
- added J1: AVR-ISP-6, Connector_PinSocket_2.54mm:PinSocket_2x03_P2.54mm_Vertical, F.Cu at (130.0, 112.0)
- added Q1: 2N7002, Package_TO_SOT_SMD:SOT-23, F.Cu at (152.7, 80.9)
- added Q2: 2N7002, Package_TO_SOT_SMD:SOT-23, F.Cu at (152.7, 86.0)
- added R10: 10k, Resistor_SMD:R_0603_1608Metric, F.Cu at (148.1, 80.1)
- added R11: 1k, Resistor_SMD:R_0603_1608Metric, F.Cu at (159.1, 90.9)
- added R12: 10k, Resistor_SMD:R_0603_1608Metric, F.Cu at (159.1, 94.5)
- added R13: 1k, Resistor_SMD:R_0603_1608Metric, F.Cu at (159.1, 98.0)
- added R14: 1k, Resistor_SMD:R_0603_1608Metric, F.Cu at (159.1, 101.3)
- added R15: 10k, Resistor_SMD:R_0603_1608Metric, F.Cu at (159.1, 104.8)
- added R16: 1k, Resistor_SMD:R_0603_1608Metric, F.Cu at (159.1, 108.4)
- added R19: R, Resistor_SMD:R_0603_1608Metric, F.Cu at (172.6, 87.6)
- added R20: R, Resistor_SMD:R_0603_1608Metric, F.Cu at (174.5, 87.6)
- added R21: R, Resistor_SMD:R_0603_1608Metric, F.Cu at (140.6, 87.4)
- added R22: R, Resistor_SMD:R_0603_1608Metric, F.Cu at (143.1, 87.4)
- added R23: R, Resistor_SMD:R_0603_1608Metric, F.Cu at (138.0, 87.4)
- added R24: R, Resistor_SMD:R_0603_1608Metric, F.Cu at (158.6, 117.6)
- added R25: R, Resistor_SMD:R_0603_1608Metric, F.Cu at (135.5, 87.4)
- added R26: R, Resistor_SMD:R_0603_1608Metric, F.Cu at (172.0, 118.3)
- added R4: 1k, Resistor_SMD:R_0603_1608Metric, F.Cu at (137.0, 98.4)
- added R5: 10k, Resistor_SMD:R_0603_1608Metric, F.Cu at (147.1, 82.7)
- added SW1: SW_Push, Button_Switch_THT:SW_PUSH_6mm, F.Cu at (129.1, 106.3)
- added U2: EL817, Package_DIP:DIP-4_W7.62mm, F.Cu at (168.8, 118.1)
- added U3: ST485EBDR, Package_SO:SOIC-8_3.9x4.9mm_P1.27mm, F.Cu at (153.0, 95.5)
- added U4: ST485EBDR, Package_SO:SOIC-8_3.9x4.9mm_P1.27mm, F.Cu at (153.2, 102.7)
- added U5: ST485EBDR, Package_SO:SOIC-8_3.9x4.9mm_P1.27mm, F.Cu at (167.5, 82.6)
- added U6: ST485EBDR, Package_SO:SOIC-8_3.9x4.9mm_P1.27mm, F.Cu at (160.5, 82.5)
- added Y1: 16MHz, Crystal:Crystal_HC49-4H_Vertical, F.Cu at (141.0, 105.5)
- D1: value 1N4001 -> BAT54CW; footprint Diode_THT:D_DO-41_SOD81_P3.81mm_Vertical_KathodeUp -> Package_TO_SOT_SMD:SOT-23
- R1, R2, R7, R8, R9: value R -> 10k
- R3, R6: value R -> 1k
- U1: value MAX489E -> ATmega328P-AU; footprint Package_SO:SOIC-14_3.9x8.7mm_P1.27mm -> Package_QFP:TQFP-32_7x7mm_P0.8mm
- moved R1 31.1 mm to (141.7, 120.4), turned to 0 degrees
- moved R8 30.7 mm to (148.1, 85.2), turned to 0 degrees
- moved D1 27.5 mm to (145.9, 94.4)
- moved R7 22.2 mm to (148.1, 87.2), turned to 0 degrees
- moved R3 19.5 mm to (137.0, 96.5), turned to 0 degrees
- moved R17 17.7 mm to (161.6, 111.1), turned to 180 degrees
- moved R9 16.6 mm to (152.7, 90.0), turned to 0 degrees
- moved R6 16.0 mm to (166.4, 111.9)
- moved U1 15.6 mm to (148.6, 114.2), turned to 270 degrees
- moved R2 15.4 mm to (148.1, 89.8)
- moved J3 12.0 mm to (168.9, 100.2)
- moved J2 9.91 mm to (130.3, 87.2)
- moved R18 7.75 mm to (161.8, 88.9), turned to 180 degrees
- renumbered J3 to J2, J1 to J3, R4 to R17, R5 to R18
Connections:
- D1 pad 2: 5V -> Net-(D1-Pad1)
- J2 pad 2: 5V -> +5V
- J3 pad 1: Net-(J1-Pad1) -> Net-(J3-Pad1)
- J3 pad 2: Net-(J1-Pad2) -> Net-(J3-Pad2)
- J3 pad 3: Net-(J1-Pad3) -> Net-(J3-Pad3)
- J3 pad 6: Net-(J1-Pad6) -> Net-(J3-Pad6)
- J3 pad 7: Net-(D1-Pad1) -> +5V
- J3 pad SH: GND -> (no net)
- P1 pad 5: 5V -> +5V
- P2 pad 5: /A4(SDA) -> (no net)
- P2 pad 6: /A5(SCL) -> (no net)
- P3 pad 1: /A5(SCL) -> (no net)
- P3 pad 2: /A4(SDA) -> (no net)
- R1 pad 1: /sense+ -> /CopRST
- R1 pad 2: Net-(OC1-Pad1) -> +5V
- R2 pad 1: 5V -> /driveB
- R2 pad 2: Net-(OC1-Pad7) -> GND
- R3 pad 1: /sense+ -> Net-(R3-Pad1)
- R3 pad 2: Net-(OC1-Pad4) -> Net-(C3-Pad1)
- R6 pad 1: /sense+B -> Net-(R6-Pad1)
- R6 pad 2: Net-(OC2-Pad1) -> /sense+
- R7 pad 1: /sense+B -> /driveInhibit
- R7 pad 2: Net-(OC2-Pad4) -> Net-(Q1-Pad1)
- R8 pad 1: /sense+B -> +5V
- R8 pad 2: Net-(J2-Pad12) -> Net-(Q1-Pad1)
- R9 pad 1: /sense+B -> /driveB
- U1 pad 10: Net-(J1-Pad3) -> Net-(R4-Pad1)
- U1 pad 11: Net-(J1-Pad1) -> Net-(R3-Pad1)
- U1 pad 12: Net-(J1-Pad2) -> Net-(R25-Pad2)
- U1 pad 13: (no net) -> Net-(SW1-Pad1)
- U1 pad 14: 5V -> (no net)
- U1 pad 2: /1(Tx) -> (no net)
- U1 pad 3: Net-(OC1-Pad7) -> GND
- U1 pad 4: 5V -> +5V
- U1 pad 5: /0(Rx) -> GND
- U1 pad 6: GND -> +5V
- U1 pad 7: GND -> Net-(C1-Pad2)
- U1 pad 8: (no net) -> Net-(C2-Pad1)
- U1 pad 9: Net-(J1-Pad6) -> (no net)
Routing:
- net +5V: track 0.00 -> 193.0 mm, vias 0 -> 6
- net 5V: track 71.6 -> 0.00 mm, vias 1 -> 0
- net /driveA: track 0.00 -> 67.8 mm, vias 0 -> 3
- net /driveB: track 0.00 -> 63.0 mm, vias 0 -> 4
- net Net-(J1-Pad1): track 52.3 -> 0.00 mm, vias 1 -> 0
- net Net-(D1-Pad1): track 57.8 -> 5.57 mm
- net Net-(OC1-Pad7): track 50.1 -> 0.00 mm
- net Net-(J1-Pad3): track 47.2 -> 0.00 mm
- net GND: track 0.00 -> 46.9 mm, vias 0 -> 11
- net /sense-B: track 45.5 -> 0.00 mm
- net Net-(J3-Pad3): track 0.00 -> 43.2 mm, vias 0 -> 2
- net Net-(J1-Pad2): track 43.1 -> 0.00 mm, vias 1 -> 0
- net /driveInhibit: track 0.00 -> 41.5 mm, vias 0 -> 2
- net Net-(J3-Pad6): track 0.00 -> 40.2 mm, vias 0 -> 2
- net Net-(J1-Pad6): track 39.4 -> 0.00 mm, vias 1 -> 0
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Other:
- board text added: "B T A"
- board text added: "INIT"
- board text added: "ISP"
- board text added: "RS485"
- board text added: "Rx Tx"
- board text removed: "1"
