File: pcbs/interface/interface.kicad_pcb (KiCad board)
At the start: 2 copper layers, 85.1 x 62.9 mm, 32 parts, among them J1 Conn_01x04, J2 AVR-ISP-6, J3 Conn_02x08_Odd_Even, J4 RJ45_LED_Shielded, J5 Conn_02x08_Odd_Even, J6 Conn_02x08_Odd_Even, J7 Conn_02x08_Odd_Even, U1 ATmega328P-AU, U10 74HC595, U2 MAX488E, U3 4021, U4 4021, U5 74HC595, U6 74HC595, U7 74HC595, U8 74HC595, U9 74HC595, Y1 16MHz

Commit message: revision b of boards
Parts:
- C3: footprint Capacitor_THT:C_Radial_D8.0mm_H11.5mm_P3.50mm -> Capacitor_THT:CP_Radial_D8.0mm_P3.50mm
Connections:
- R8 pad 1: Net-(J4-Pad2) -> Net-(J4-Pad1)
- R8 pad 2: Net-(J4-Pad1) -> Net-(J4-Pad2)
- U2 pad 7: Net-(J4-Pad2) -> Net-(J4-Pad1)
- U2 pad 8: Net-(J4-Pad1) -> Net-(J4-Pad2)
Routing:
- net 5V: track 348.7 -> 354.0 mm
- net Net-(J4-Pad3): track 26.4 -> 22.9 mm, vias 0 -> 1
- net GND: track 54.0 -> 52.4 mm, vias 14 -> 13
- net ~OE: track 113.7 -> 114.8 mm
- net Net-(J4-Pad2): track 15.5 -> 14.5 mm, vias 0 -> 1
- net Net-(J4-Pad1): track 18.6 -> 17.7 mm
- net LATCH_OUT: track 118.3 -> 118.9 mm
