File: pcbs/interface/networking.sch (KiCad schematic (older format))
At the start: 5 parts, among them J4 RJ45_LED_Shielded, U2 MAX488E

Commit message: revision b of boards
Connections:
- net at R8.2, U2.8 (A): now also J4.2; no longer J4.1
- net at R8.1, U2.7 (B): now also J4.1; no longer J4.2
Changed lines of the file:
@@
 Connection ~ 4400 2500
-Wire Wire Line
-	4400 2500 6000 2500
 Wire Wire Line
 	4700 2350 4700 2600
 Connection ~ 4700 2600
 Wire Wire Line
-	4700 2600 6000 2600
+	4700 2600 5400 2600
 Text GLabel 5800 3150 0    50   Input ~ 0
 5V
@@
 Text GLabel 7100 2500 2    50   Input ~ 0
 5V
+Wire Wire Line
+	5400 2600 5400 2500
+Wire Wire Line
+	4400 2500 5350 2500
+Wire Wire Line
+	5400 2500 6000 2500
+Wire Wire Line
+	5450 2600 5450 2550
+Wire Wire Line
+	5450 2550 5350 2550
+Wire Wire Line
+	5350 2550 5350 2500
+Wire Wire Line
+	5450 2600 6000 2600
 $EndSCHEMATC
