File: pcbs/switch_decoder/decoder.sch (KiCad schematic (older format))
At the start: 18 parts, among them J1 Screw_Terminal_01x06, J2 AVR-ISP-6, J3 Screw_Terminal_01x06, SW1 SW_DIP_x06, U1 ATmega328P-AU, U10 74HC595, U2 74HC595, Y1 16MHz

Commit message: revision b of boards
Parts:
- C3: footprint Capacitor_THT:C_Radial_D8.0mm_H11.5mm_P3.50mm -> Capacitor_THT:CP_Radial_D8.0mm_P3.50mm
Changed lines of the file:
@@
 F 0 "C3" H 3968 1446 50  0000 L CNN
 F 1 "220uF" H 3968 1355 50  0000 L CNN
-F 2 "Capacitor_THT:C_Radial_D8.0mm_H11.5mm_P3.50mm" H 3888 1250 50  0001 C CNN
+F 2 "Capacitor_THT:CP_Radial_D8.0mm_P3.50mm" H 3888 1250 50  0001 C CNN
 F 3 "~" H 3850 1400 50  0001 C CNN
 	1    3850 1400
