File: pcbs/servo_driver/servo_driver.kicad_pcb (KiCad board)
At the start: 2 copper layers, 44.4 x 33.7 mm, 19 parts, among them J1 Screw_Terminal_01x04, J2 Conn_01x04_Male, J3 AVR-ISP-6, SW1 SW_Push, U1 ATmega328P-AU, Y1 16MHz

Commit message: servo driver rev. A
Parts:
- added C7: 100nF, Capacitor_SMD:C_0603_1608Metric, F.Cu at (135.3, 94.6)
- added C8: 100nF, Capacitor_SMD:C_0603_1608Metric, F.Cu at (133.3, 98.4)
- added LED3: LED, LED_SMD:LED_0603_1608Metric, F.Cu at (114.3, 107.3)
- added R4: 10k, Resistor_SMD:R_0603_1608Metric, F.Cu at (114.3, 109.2)
- J1: renamed from J3; footprint Connector_PinSocket_2.54mm:PinSocket_2x03_P2.54mm_Vertical -> Connector_IDC:IDC-Header_2x03_P2.54mm_Vertical
- moved C2 28.3 mm to (123.2, 83.2), turned to 180 degrees
- moved C1 27.4 mm to (128.3, 83.2), turned to 180 degrees
- moved J1 22.5 mm to (122.6, 108.6), turned to 90 degrees
- moved Y1 19.8 mm to (128.3, 87.0), turned to 180 degrees
- moved R3 13.2 mm to (131.3, 101.0), turned to 180 degrees
- moved C5 6.34 mm to (118.1, 94.1), turned to 90 degrees
- moved C6 4.76 mm to (118.1, 98.9), turned to 270 degrees
- moved C3 2.66 mm to (119.4, 90.2), turned to 270 degrees
- moved U1 2.29 mm to (125.9, 96.5), turned to 270 degrees
- moved J2 1.91 mm to (112.4, 94.6)
- moved C4 0.63 mm to (114.3, 87.0)
- renumbered J1 to J2, J2 to J3, R2 to R1, R3 to R2, R1 to R3
Connections:
- net Net-(C1-Pad1) renamed /XTAL1
- net Net-(C2-Pad2) renamed /XTAL2
- J1 pad 1: MISO -> 5V
- J1 pad 2: 5V -> MISO
- J1 pad 3: SCK -> MOSI
- J1 pad 4: MOSI -> SCK
- J1 pad 5: ~RST -> GND
- J1 pad 6: GND -> ~RST
- J2 pad 2: sig_A -> 5V
- J2 pad 3: sig_B -> sig_A
- J2 pad 4: 5V -> sig_B
- U1 pad 1: sig_A -> (no net)
- U1 pad 10: servo -> (no net)
- U1 pad 11: sig_T -> (no net)
- U1 pad 12: (no net) -> sig_A
- U1 pad 13: (no net) -> sig_B
- U1 pad 14: LED_A -> LED_C
- U1 pad 2: sig_B -> (no net)
- U1 pad 23: rv1 -> (no net)
- U1 pad 24: rv2 -> LED_B
- U1 pad 25: (no net) -> rv2
- U1 pad 26: (no net) -> servo
- U1 pad 27: (no net) -> sig_T
- U1 pad 28: (no net) -> rv1
- U1 pad 30: (no net) -> LED_A
- U1 pad 9: LED_B -> (no net)
Routing:
- net LED_C: track 0.00 -> 16.7 mm
- net rv2: track 29.7 -> 13.7 mm, vias 2 -> 0
- net rv1: track 18.4 -> 11.7 mm, vias 2 -> 0
- net GND: track 18.6 -> 24.6 mm, vias 1 -> 8
- net sig_A: track 18.9 -> 13.2 mm
- net LED_B: track 13.2 -> 18.3 mm, vias 0 -> 2
- net sig_B: track 17.8 -> 14.7 mm
- net SCK: track 8.91 -> 6.16 mm
- net servo: track 17.3 -> 19.8 mm
- net 5V: track 119.0 -> 121.3 mm, vias 4 -> 3
- net Net-(LED3-Pad2): track 0.00 -> 1.92 mm
- net sig_T: track 11.4 -> 13.2 mm
- net MOSI: track 16.9 -> 15.5 mm
- net LED_A: track 10.8 -> 12.2 mm
- net MISO: track 10.9 -> 10.4 mm
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Other:
- board text added: "SERVO SWITCH CONTROL Rev.A"
